File: SPGA_PU/MCU.kicad_sch (KiCad schematic)
At the start: 5 parts, among them U19 ESP32-S3-WROOM-1

Commit message: I dunno
Changed lines of the file:
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@@
 	(global_label "FRET_1_STR_G"
 		(shape input)
-		(at 280.67 91.44 180)
-		(fields_autoplaced yes)
-		(effects
-			(font
-				(size 1 1)
-				(color 0 0 0 1)
-			)
-			(justify right)
-		)
-		(property "Intersheetrefs" "${INTERSHEET_REFS}"
-			(at 267.8435 91.44 0)
+		(at 254 69.85 180)
+		(fields_autoplaced yes)
+		(effects
+			(font
+				(size 1 1)
+				(color 0 0 0 1)
+			)
+			(justify right)
+		)
+		(property "Intersheetrefs" "${INTERSHEET_REFS}"
+			(at 241.1735 69.85 0)
 			(effects
 				(font
@@
 	(global_label "CLK_SR"
 		(shape input)
-		(at 280.67 109.22 180)
-		(fields_autoplaced yes)
-		(effects
-			(font
-				(size 1 1)
-				(color 0 0 0 1)
-			)
-			(justify right)
-		)
-		(property "Intersheetrefs" "${INTERSHEET_REFS}"
-			(at 272.7959 109.22 0)
+		(at 254 87.63 180)
+		(fields_autoplaced yes)
+		(effects
+			(font
+				(size 1 1)
+				(color 0 0 0 1)
+			)
+			(justify right)
+		)
+		(property "Intersheetrefs" "${INTERSHEET_REFS}"
+			(at 246.1259 87.63 0)
 			(effects
 				(font
@@
 	(global_label "FRET_1_STR_D"
 		(shape input)
-		(at 280.67 93.98 180)
-		(fields_autoplaced yes)
-		(effects
-			(font
-				(size 1 1)
-				(color 0 0 0 1)
-			)
-			(justify right)
-		)
-		(property "Intersheetrefs" "${INTERSHEET_REFS}"
-			(at 267.8435 93.98 0)
+		(at 254 72.39 180)
+		(fields_autoplaced yes)
+		(effects
+			(font
+				(size 1 1)
+				(color 0 0 0 1)
+			)
+			(justify right)
+		)
+		(property "Intersheetrefs" "${INTERSHEET_REFS}"
+			(at 241.1735 72.39 0)
 			(effects
 				(font
@@
 	(global_label "FRET_1_STR_A"
 		(shape input)
-		(at 280.67 96.52 180)
-		(fields_autoplaced yes)
-		(effects
-			(font
-				(size 1 1)
-				(color 0 0 0 1)
-			)
-			(justify right)
-		)
-		(property "Intersheetrefs" "${INTERSHEET_REFS}"
-			(at 267.9864 96.52 0)
+		(at 254 74.93 180)
+		(fields_autoplaced yes)
+		(effects
+			(font
+				(size 1 1)
+				(color 0 0 0 1)
+			)
+			(justify right)
+		)
+		(property "Intersheetrefs" "${INTERSHEET_REFS}"
+			(at 241.3164 74.93 0)
 			(effects
 				(font
@@
 	(global_label "LATCH_SR"
 		(shape input)
-		(at 280.67 106.68 180)
-		(fields_autoplaced yes)
-		(effects
-			(font
-				(size 1 1)
-				(color 0 0 0 1)
-			)
-			(justify right)
-		)
-		(property "Intersheetrefs" "${INTERSHEET_REFS}"
-			(at 271.1293 106.68 0)
+		(at 254 85.09 180)
+		(fields_autoplaced yes)
+		(effects
+			(font
+				(size 1 1)
+				(color 0 0 0 1)
+			)
+			(justify right)
+		)
+		(property "Intersheetrefs" "${INTERSHEET_REFS}"
+			(at 244.4593 85.09 0)
 			(effects
 				(font
@@
 	(global_label "FRET_1_STR_E"
 		(shape input)
-		(at 280.67 99.06 180)
-		(fields_autoplaced yes)
-		(effects
-			(font
-				(size 1 1)
-				(color 0 0 0 1)
-			)
-			(justify right)
-		)
-		(property "Intersheetrefs" "${INTERSHEET_REFS}"
-			(at 267.9387 99.06 0)
+		(at 254 77.47 180)
+		(fields_autoplaced yes)
+		(effects
+			(font
+				(size 1 1)
+				(color 0 0 0 1)
+			)
+			(justify right)
+		)
+		(property "Intersheetrefs" "${INTERSHEET_REFS}"
+			(at 241.2687 77.47 0)
 			(effects
 				(font
@@
 	(global_label "INPUT_FRET_1"
 		(shape input)
-		(at 280.67 104.14 180)
-		(fields_autoplaced yes)
-		(effects
-			(font
-				(size 1 1)
-				(color 0 0 0 1)
-			)
-			(justify right)
-		)
-		(property "Intersheetrefs" "${INTERSHEET_REFS}"
-			(at 267.9864 104.14 0)
+		(at 254 82.55 180)
+		(fields_autoplaced yes)
+		(effects
+			(font
+				(size 1 1)
+				(color 0 0 0 1)
+			)
+			(justify right)
+		)
+		(property "Intersheetrefs" "${INTERSHEET_REFS}"
+			(at 241.3164 82.55 0)
 			(effects
 				(font
@@
 	(global_label "FRET_1_STR_EH"
 		(shape input)
-		(at 280.67 101.6 180)
-		(fields_autoplaced yes)
-		(effects
-			(font
-				(size 1 1)
-				(color 0 0 0 1)
-			)
-			(justify right)
-		)
-		(property "Intersheetrefs" "${INTERSHEET_REFS}"
-			(at 266.8911 101.6 0)
-			(effects
-				(font
+		(at 254 80.01 180)
+		(fields_autoplaced yes)
+		(effects
+			(font
+				(size 1 1)
+				(color 0 0 0 1)
+			)
+			(justify right)
+		)
+		(property "Intersheetrefs" "${INTERSHEET_REFS}"
+			(at 240.2211 80.01 0)
+			(effects
+				(font

Commit message: thibgs
Parts:
- added C1, C7: 100nF, Capacitor_SMD:C_0805_2012Metric_Pad1.18x1.45mm_HandSolder, symbol Device:C
- added D1: D_Schottky, Diode_SMD:D_1206_3216Metric_Pad1.42x1.75mm_HandSolder, symbol Device:D_Schottky
- added F1: Polyfuse, Fuse:Fuse_0805_2012Metric, symbol Device:Polyfuse
- added J1: USB_TypeC, sumec_brd:HRO_TYPE-C-31-M-12, symbol sumec_sch_lib:USB_TypeC
- added R32: 100k, Resistor_SMD:R_0805_2012Metric_Pad1.20x1.40mm_HandSolder, symbol Device:R
- added R33, R34: 15R, Resistor_SMD:R_0805_2012Metric_Pad1.20x1.40mm_HandSolder, symbol Device:R
- added U5: USBLC6-2SC6, Package_TO_SOT_SMD:TSOT-23-6_HandSoldering, symbol sumec_library:USBLC6-2SC6
Connections:
- net GND: now also C1.1, C7.2, J1.A1_B12 (GND), J1.B1_A12 (GND), R32.2, U5.2
- new net: R33.2, U5.1
- new net: R34.2, U5.3
- new net: D1.2 (A), F1.1
- new net: F1.2, J1.A4_B9 (VBUS), J1.B4_A9 (VBUS)
- new net +5V: C7.1, D1.1 (K), U5.5
- new net D+: U5.6
- new net D+ IN: J1.A6 (DP1), J1.B6 (DP2), R33.1
- new net D-: U5.4
- new net D- IN: J1.A7 (DN1), J1.B7 (DN2), R34.1
- new net SHLD: C1.2, J1.S1 (SHIELD), J1.S2 (SHIELD), J1.S3 (SHIELD), J1.S4 (SHIELD), R32.1
- no-connect marks 4 -> 8
Other:
- note added: "ESD PROTECTION"
- note added: "GPIO USB 20 D+ (green) 19 D- (white) GND GND (black) VBUS +5V (red)"
- note added: "USB"
- note added: "USB CONNECTOR"
- note added: "USB Type-C Connector Data transfer USB connector connected to ESP32 using CDC method"
