File: SPGA_PU/MECHANICS.kicad_sch (KiCad schematic)
At the start: 15 parts, among them SW2 SW_Push, SW3 SW_Push, SW4 SW_Push, SW5 SW_Push

Commit message: thibgs
Parts:
- added C12: 10uF, Capacitor_Tantalum_SMD:CP_EIA-3216-18_Kemet-A_Pad1.58x1.35mm_HandSolder, symbol Device:C_Polarized
- added C13: 100nF, Capacitor_SMD:C_0805_2012Metric_Pad1.18x1.45mm_HandSolder, symbol Device:C
- added J4: MEM2067-02-180-00-A_REVB, Schrack_brd:MICRO_SD_CARD, symbol SchrackThingy_library:MEM2067-02-180-00-A_REVB
- added R31: 10k, Resistor_SMD:R_0805_2012Metric_Pad1.20x1.40mm_HandSolder, symbol Device:R
Connections:
- net +3V3: now also C12.1, C13.1, J4.4 (VDD), R31.2
- net GND: now also C12.2, C13.2, J4.10 (SHIELD), J4.11 (SHIELD), J4.12 (SHIELD), J4.6 (VSS), J4.9 (SHIELD)
- new net IO04_MISO: J4.7 (DAT0)
- new net IO05_CLK: J4.5 (CLK)
- new net IO06_MOSI: J4.3 (CMD)
- new net IO07_~{CS}: J4.2 (CD/DAT3), R31.1
- no-connect marks 0 -> 2
Other:
- note added: "MICRO SD"
