File: SPGA_PU/SPGA_PU.kicad_sch (KiCad schematic)
At the start: 10 parts

Commit message: I dunno
Other:
- sheet FRETBOARD renamed FRET POSITION
- sheet FRET POSITION: file FRETBOARD.kicad_sch -> FRET_POSITION.kicad_sch
